File: energymonitor-arduino-basic/energymonitor-arduino-basic.sch (KiCad schematic (older format))
At the start: 15 parts

Commit message: Add switched dc jack, add arduino, add LCD I2C
Parts:
- removed J?: Conn_01x05_Female, symbol Connector:Conn_01x05_Female
- added A1: Arduino_Nano_v3.x, Module:Arduino_Nano, symbol MCU_Module:Arduino_Nano_v3.x
- added J3: Conn_01x04_Male, symbol Connector:Conn_01x04_Male
- J1: renamed from J?; symbol Connector:Barrel_Jack -> Connector:Barrel_Jack_Switch
- J4: renamed from J?; symbol Connector:Conn_01x03_Female -> Connector:Conn_01x03_Male
- gave numbers to parts that had none: 10
Connections:
- net +5V: now also A1.27 (+5V), J3.2 (Pin_2)
- net 1wire-bus: now also J4.3 (Pin_3), A1.5 (D2); no longer J4.1 (Pin_1)
- net GND: now also J4.1 (Pin_1), A1.29 (GND), A1.4 (GND), J3.1 (Pin_1); no longer J4.3 (Pin_3)
- net current-sense: now also A1.21 (A2)
- net voltage-sense: now also A1.22 (A3)
- new net SCL: A1.24 (A5), J3.4 (Pin_4)
- new net SDA: A1.23 (A4), J3.3 (Pin_3)
- no-connect marks 5 -> 6
Other:
- note added: "LCD I2C"
- note added: "Midpoint buffer"
- note added: "SCL"
- note added: "SDA"
Changed lines of the file:
@@
 $EndDescr
 $Comp
-L Connector:Conn_01x05_Female J?
-U 1 1 62606ACB
-P 7150 1500
-F 0 "J?" H 7178 1476 50  0000 L CNN
-F 1 "Conn_01x05_Female" H 7178 1385 50  0000 L CNN
-F 2 "" H 7150 1500 50  0001 C CNN
-F 3 "~" H 7150 1500 50  0001 C CNN
-	1    7150 1500
-	1    0    0    -1
-$EndComp
-$Comp
-L power:+5V #PWR0101
-U 1 1 626076B4
-P 6150 1050
-F 0 "#PWR0101" H 6150 900 50  0001 C CNN
-F 1 "+5V" H 6165 1223 50  0000 C CNN
-F 2 "" H 6150 1050 50  0001 C CNN
-F 3 "" H 6150 1050 50  0001 C CNN
-	1    6150 1050
-	1    0    0    -1
-$EndComp
-$Comp
-L power:GND #PWR0102
-U 1 1 62607C1A
-P 6150 2550
-F 0 "#PWR0102" H 6150 2300 50  0001 C CNN
-F 1 "GND" H 6155 2377 50  0000 C CNN
-F 2 "" H 6150 2550 50  0001 C CNN
-F 3 "" H 6150 2550 50  0001 C CNN
-	1    6150 2550
-	1    0    0    -1
-$EndComp
-Wire Wire Line
-	6950 1300 6150 1300
-Wire Wire Line
-	6150 1300 6150 1050
-Wire Wire Line
-	6950 1400 6150 1400
-Wire Wire Line
-	6150 1400 6150 2550
-$Comp
-L Connector:AudioJack3_Ground_SwitchTR J?
+L Connector:AudioJack3_Ground_SwitchTR J2
 U 1 1 6260899F
 P 2250 1400
-F 0 "J?" H 2232 1725 50  0000 C CNN
+F 0 "J2" H 2232 1725 50  0000 C CNN
 F 1 "AudioJack3_Ground_SwitchTR" H 2232 1634 50  0000 C CNN
 F 2 "" H 2250 1400 50  0001 C CNN
@@
 	2250 2150 2250 2000
 $Comp
-L Device:R R?
+L Device:R R3
 U 1 1 6260C8A0
 P 2800 1450
-F 0 "R?" H 2870 1496 50  0000 L CNN
+F 0 "R3" H 2870 1496 50  0000 L CNN
 F 1 "33R" H 2870 1405 50  0000 L CNN
 F 2 "Resistor_THT:R_Axial_DIN0207_L6.3mm_D2.5mm_P10.16mm_Horizontal" V 2730 1450 50  0001 C CNN
@@
 	2800 1300 3900 1300
 Connection ~ 2800 1300
-Text Label 6750 1500 2    50   ~ 0
-current-sense
-Wire Wire Line
-	6750 1500 6950 1500
-Text Label 6750 1600 2    50   ~ 0
-voltage-sense
-Wire Wire Line
-	6950 1600 6750 1600
-$Comp
-L Connector:Barrel_Jack J?
+$Comp
+L Connector:Barrel_Jack_Switch J1
 U 1 1 6262B60D
 P 2100 3550
-F 0 "J?" H 2157 3875 50  0000 C CNN
+F 0 "J1" H 2157 3875 50  0000 C CNN
 F 1 "Barrel_Jack" H 2157 3784 50  0000 C CNN
 F 2 "" H 2150 3510 50  0001 C CNN
@@
 $EndComp
 $Comp
-L Device:R R?
+L Device:R R5
 U 1 1 6262BC5E
 P 9400 4450
-F 0 "R?" V 9193 4450 50  0000 C CNN
+F 0 "R5" V 9193 4450 50  0000 C CNN
 F 1 "10k" V 9284 4450 50  0000 C CNN
 F 2 "Resistor_THT:R_Axial_DIN0207_L6.3mm_D2.5mm_P10.16mm_Horizontal" V 9330 4450 50  0001 C CNN
@@
 $EndComp
 $Comp
-L Device:R R?
+L Device:R R6
 U 1 1 6262C6E4
 P 9900 4450
-F 0 "R?" V 9693 4450 50  0000 C CNN
+F 0 "R6" V 9693 4450 50  0000 C CNN
 F 1 "10k" V 9784 4450 50  0000 C CNN
 F 2 "Resistor_THT:R_Axial_DIN0207_L6.3mm_D2.5mm_P10.16mm_Horizontal" V 9830 4450 50  0001 C CNN
@@
 $EndComp
 $Comp
-L Device:CP C?
+L Device:CP C2
 U 1 1 6262CCE6
 P 9650 4750
-F 0 "C?" H 9768 4796 50  0000 L CNN
+F 0 "C2" H 9768 4796 50  0000 L CNN
 F 1 "10uf" H 9768 4705 50  0000 L CNN
 F 2 "" H 9688 4600 50  0001 C CNN
@@
 voltage-sense
 $Comp
-L Device:R R?
+L Device:R R1
 U 1 1 62631A9B
 P 2750 3450
-F 0 "R?" V 2543 3450 50  0000 C CNN
+F 0 "R1" V 2543 3450 50  0000 C CNN
 F 1 "100k" V 2634 3450 50  0000 C CNN
 F 2 "Resistor_THT:R_Axial_DIN0207_L6.3mm_D2.5mm_P10.16mm_Horizontal" V 2680 3450 50  0001 C CNN
@@
 $EndComp
 $Comp
-L Device:R R?
+L Device:R R2
 U 1 1 62631FC5
 P 2750 3650
-F 0 "R?" V 2543 3650 50  0000 C CNN
+F 0 "R2" V 2543 3650 50  0000 C CNN
 F 1 "10k" V 2634 3650 50  0000 C CNN
 F 2 "Resistor_THT:R_Axial_DIN0207_L6.3mm_D2.5mm_P10.16mm_Horizontal" V 2680 3650 50  0001 C CNN
@@
 Text Notes 2850 3800 0    50   ~ 0
 Step down voltage divider
-Text Label 6750 1700 2    50   ~ 0
-1wire-bus
-Wire Wire Line
-	6950 1700 6750 1700
-$Comp
-L Connector:Conn_01x03_Female J?
+$Comp
+L Connector:Conn_01x03_Male J4
 U 1 1 6261A3BF
 P 5550 3550
-F 0 "J?" H 5442 3225 50  0000 C CNN
+F 0 "J4" H 5442 3225 50  0000 C CNN
 F 1 "Conn_01x03_Female" H 5442 3316 50  0000 C CNN
 F 2 "" H 5550 3550 50  0001 C CNN
 F 3 "~" H 5550 3550 50  0001 C CNN
 	1    5550 3550
-	-1   0    0    1
+	1    0    0    -1
 $EndComp
 $Comp
@@
 1wire-bus
 $Comp
-L Device:R R?
+L Device:R R4
 U 1 1 6261CDC5
 P 6800 3550
-F 0 "R?" V 6593 3550 50  0000 C CNN
+F 0 "R4" V 6593 3550 50  0000 C CNN
 F 1 "4k7" V 6684 3550 50  0000 C CNN
 F 2 "Resistor_THT:R_Axial_DIN0207_L6.3mm_D2.5mm_P10.16mm_Horizontal" V 6730 3550 50  0001 C CNN
@@
 	6550 3350 6550 3550
 $Comp
-L Device:C C?
+L Device:C C1
 U 1 1 6263CCEC
 P 6300 3350
-F 0 "C?" V 6048 3350 50  0000 C CNN
+F 0 "C1" V 6048 3350 50  0000 C CNN
 F 1 "C" V 6139 3350 50  0000 C CNN
 F 2 "" H 6338 3200 50  0001 C CNN
@@
 Text Notes 1750 3850 0    50   ~ 0
 9v AC
-Text Notes 5050 3800 0    50   ~ 0
+Text Notes 5450 3300 0    50   ~ 0
 DS18B20
 $Comp
-L Amplifier_Operational:LM358 U?
+L Amplifier_Operational:LM358 U1
 U 1 1 6278D4CE
 P 6350 4450
-F 0 "U?" H 6350 4817 50  0000 C CNN
+F 0 "U1" H 6350 4817 50  0000 C CNN
 F 1 "LM358" H 6350 4726 50  0000 C CNN
 F 2 "" H 6350 4450 50  0001 C CNN
@@
 $EndComp
 $Comp
-L Amplifier_Operational:LM358 U?
+L Amplifier_Operational:LM358 U1
 U 2 1 6278EB53
 P 3750 6350
-F 0 "U?" H 3750 6717 50  0000 C CNN
+F 0 "U1" H 3750 6717 50  0000 C CNN
 F 1 "LM358" H 3750 6626 50  0000 C CNN
 F 2 "" H 3750 6350 50  0001 C CNN
@@
 $EndComp
 $Comp
-L Amplifier_Operational:LM358 U?
+L Amplifier_Operational:LM358 U1
 U 3 1 6278FD5E
 P 8750 2250
-F 0 "U?" H 8708 2296 50  0000 L CNN
+F 0 "U1" H 8708 2296 50  0000 L CNN
 F 1 "LM358" H 8708 2205 50  0000 L CNN
 F 2 "" H 8750 2250 50  0001 C CNN
@@
 	5800 4550 6050 4550
 $Comp
-L power:GND #PWR?
+L power:GND #PWR0101
 U 1 1 627A363E
 P 8650 2700
-F 0 "#PWR?" H 8650 2450 50  0001 C CNN
+F 0 "#PWR0101" H 8650 2450 50  0001 C CNN
 F 1 "GND" H 8655 2527 50  0000 C CNN
 F 2 "" H 8650 2700 50  0001 C CNN
@@
 $EndComp
 $Comp
-L power:+5V #PWR?
+L power:+5V #PWR0102
 U 1 1 627A3F4D
 P 8650 1800
-F 0 "#PWR?" H 8650 1650 50  0001 C CNN
+F 0 "#PWR0102" H 8650 1650 50  0001 C CNN
 F 1 "+5V" H 8665 1973 50  0000 C CNN
 F 2 "" H 8650 1800 50  0001 C CNN
@@
 Wire Wire Line
 	2500 3650 2600 3650
+$Comp
+L MCU_Module:Arduino_Nano_v3.x A1
+U 1 1 6266E5DC
+P 9950 2150
+F 0 "A1" H 9950 1061 50  0000 C CNN
+F 1 "Arduino_Nano_v3.x" H 9950 970 50  0000 C CNN
+F 2 "Module:Arduino_Nano" H 9950 2150 50  0001 C CIN
+F 3 "http://www.mouser.com/pdfdocs/Gravitech_Arduino_Nano3_0.pdf" H 9950 2150 50  0001 C CNN
+	1    9950 2150
+	1    0    0    -1
+$EndComp
+Text Label 10550 2550 0    50   ~ 0
+SDA
+Text Label 10550 2650 0    50   ~ 0
+SCL
+Text Label 10550 2450 0    50   ~ 0
+voltage-sense
+Text Label 10550 2350 0    50   ~ 0
+current-sense
+Wire Wire Line
+	10450 2350 10550 2350
+Wire Wire Line
+	10550 2450 10450 2450
+Wire Wire Line
+	10550 2550 10450 2550
+Wire Wire Line
+	10450 2650 10550 2650
+Text Label 9350 1750 2    50   ~ 0
+1wire-bus
+$Comp
+L Connector:Conn_01x04_Male J3
+U 1 1 626A410F
+P 5550 2350
+F 0 "J3" H 5658 2631 50  0000 C CNN
+F 1 "Conn_01x04_Male" H 5658 2540 50  0000 C CNN
+F 2 "" H 5550 2350 50  0001 C CNN
+F 3 "~" H 5550 2350 50  0001 C CNN
+	1    5550 2350
+	1    0    0    -1
+$EndComp
+$Comp
+L power:GND #PWR0104
+U 1 1 626AA30E
+P 6050 2150
+F 0 "#PWR0104" H 6050 1900 50  0001 C CNN
+F 1 "GND" H 6055 1977 50  0000 C CNN
+F 2 "" H 6050 2150 50  0001 C CNN
+F 3 "" H 6050 2150 50  0001 C CNN
+	1    6050 2150
+	-1   0    0    1
+$EndComp
+$Comp
+L power:+5V #PWR0105
+U 1 1 626AB822
+P 6300 2350
+F 0 "#PWR0105" H 6300 2200 50  0001 C CNN
+F 1 "+5V" V 6315 2478 50  0000 L CNN
+F 2 "" H 6300 2350 50  0001 C CNN
+F 3 "" H 6300 2350 50  0001 C CNN
+	1    6300 2350
+	0    1    1    0
+$EndComp
+Text Label 6050 2450 0    50   ~ 0
+SDA
+Text Label 6050 2550 0    50   ~ 0
+SCL
+Wire Wire Line
+	6050 2550 5750 2550
+Wire Wire Line
+	5750 2450 6050 2450
+Wire Wire Line
+	6300 2350 5750 2350
+Wire Wire Line
+	6050 2150 6050 2250
+Wire Wire Line
+	6050 2250 5750 2250
+Wire Wire Line
+	9450 1750 9350 1750
+Text Notes 5750 2000 2    50   ~ 0
+LCD I2C
+Text Notes 5450 2250 2    50   ~ 0
+GND
+Text Notes 5450 2350 2    50   ~ 0
+VCC
+Text Notes 5450 2450 2    50   ~ 0
+SDA
+Text Notes 5450 2550 2    50   ~ 0
+SCL
+Text Notes 6550 4950 2    50   ~ 0
+Midpoint buffer
+$Comp
+L power:GND #PWR0110
+U 1 1 626D2DC1
+P 10050 3500
+F 0 "#PWR0110" H 10050 3250 50  0001 C CNN
+F 1 "GND" H 10055 3327 50  0000 C CNN
+F 2 "" H 10050 3500 50  0001 C CNN
+F 3 "" H 10050 3500 50  0001 C CNN
+	1    10050 3500
+	1    0    0    -1
+$EndComp
+Wire Wire Line
+	10050 3150 10050 3450
+Wire Wire Line
+	9950 3150 9950 3450
+Wire Wire Line
+	9950 3450 10050 3450
+Connection ~ 10050 3450
+Wire Wire Line
+	10050 3450 10050 3500
+$Comp
+L power:+5V #PWR0111
+U 1 1 626D928D
+P 10150 950
+F 0 "#PWR0111" H 10150 800 50  0001 C CNN
+F 1 "+5V" H 10165 1123 50  0000 C CNN
+F 2 "" H 10150 950 50  0001 C CNN
+F 3 "" H 10150 950 50  0001 C CNN
+	1    10150 950
+	1    0    0    -1
+$EndComp
+Wire Wire Line
+	10150 950  10150 1150
+NoConn ~ 2400 3550
 $EndSCHEMATC

Commit message: Add footprints
Parts:
- C1: footprint (none) -> Capacitor_THT:C_Rect_L7.0mm_W4.5mm_P5.00mm
- C2: footprint (none) -> Capacitor_THT:CP_Radial_D5.0mm_P2.00mm
- J1: footprint (none) -> Connector_BarrelJack:BarrelJack_Wuerth_6941xx301002
- J3: footprint (none) -> Connector_PinHeader_2.54mm:PinHeader_1x04_P2.54mm_Vertical
- J4: footprint (none) -> TerminalBlock:TerminalBlock_bornier-3_P5.08mm
- U1: footprint (none) -> Package_DIP:DIP-8_W10.16mm_LongPads
Changed lines of the file:
@@
 F 0 "J1" H 2157 3875 50  0000 C CNN
 F 1 "Barrel_Jack" H 2157 3784 50  0000 C CNN
-F 2 "" H 2150 3510 50  0001 C CNN
+F 2 "Connector_BarrelJack:BarrelJack_Wuerth_6941xx301002" H 2150 3510 50  0001 C CNN
 F 3 "~" H 2150 3510 50  0001 C CNN
 	1    2100 3550
@@
 F 0 "C2" H 9768 4796 50  0000 L CNN
 F 1 "10uf" H 9768 4705 50  0000 L CNN
-F 2 "" H 9688 4600 50  0001 C CNN
+F 2 "Capacitor_THT:CP_Radial_D5.0mm_P2.00mm" H 9688 4600 50  0001 C CNN
 F 3 "~" H 9650 4750 50  0001 C CNN
 	1    9650 4750
@@
 F 0 "J4" H 5442 3225 50  0000 C CNN
 F 1 "Conn_01x03_Female" H 5442 3316 50  0000 C CNN
-F 2 "" H 5550 3550 50  0001 C CNN
+F 2 "TerminalBlock:TerminalBlock_bornier-3_P5.08mm" H 5550 3550 50  0001 C CNN
 F 3 "~" H 5550 3550 50  0001 C CNN
 	1    5550 3550
@@
 F 0 "C1" V 6048 3350 50  0000 C CNN
 F 1 "C" V 6139 3350 50  0000 C CNN
-F 2 "" H 6338 3200 50  0001 C CNN
+F 2 "Capacitor_THT:C_Rect_L7.0mm_W4.5mm_P5.00mm" H 6338 3200 50  0001 C CNN
 F 3 "~" H 6300 3350 50  0001 C CNN
 	1    6300 3350
@@
 F 0 "U1" H 6350 4817 50  0000 C CNN
 F 1 "LM358" H 6350 4726 50  0000 C CNN
-F 2 "" H 6350 4450 50  0001 C CNN
+F 2 "Package_DIP:DIP-8_W10.16mm_LongPads" H 6350 4450 50  0001 C CNN
 F 3 "http://www.ti.com/lit/ds/symlink/lm2904-n.pdf" H 6350 4450 50  0001 C CNN
 	1    6350 4450
@@
 F 0 "U1" H 3750 6717 50  0000 C CNN
 F 1 "LM358" H 3750 6626 50  0000 C CNN
-F 2 "" H 3750 6350 50  0001 C CNN
+F 2 "Package_DIP:DIP-8_W10.16mm_LongPads" H 3750 6350 50  0001 C CNN
 F 3 "http://www.ti.com/lit/ds/symlink/lm2904-n.pdf" H 3750 6350 50  0001 C CNN
 	2    3750 6350
@@
 F 0 "U1" H 8708 2296 50  0000 L CNN
 F 1 "LM358" H 8708 2205 50  0000 L CNN
-F 2 "" H 8750 2250 50  0001 C CNN
+F 2 "Package_DIP:DIP-8_W10.16mm_LongPads" H 8750 2250 50  0001 C CNN
 F 3 "http://www.ti.com/lit/ds/symlink/lm2904-n.pdf" H 8750 2250 50  0001 C CNN
 	3    8750 2250
@@
 F 0 "J3" H 5658 2631 50  0000 C CNN
 F 1 "Conn_01x04_Male" H 5658 2540 50  0000 C CNN
-F 2 "" H 5550 2350 50  0001 C CNN
+F 2 "Connector_PinHeader_2.54mm:PinHeader_1x04_P2.54mm_Vertical" H 5550 2350 50  0001 C CNN
 F 3 "~" H 5550 2350 50  0001 C CNN
 	1    5550 2350

Commit message: Use jack without GND
Parts:
- J2: symbol Connector:AudioJack3_Ground_SwitchTR -> Connector:AudioJack3_SwitchTR
Connections:
- net GND: no longer J2.G
Changed lines of the file:
@@
 $EndDescr
 $Comp
-L Connector:AudioJack3_Ground_SwitchTR J2
+L Connector:AudioJack3_SwitchTR J2
 U 1 1 6260899F
 P 2250 1400
@@
 L power:GND #PWR0103
 U 1 1 6260B66F
-P 2250 2150
-F 0 "#PWR0103" H 2250 1900 50  0001 C CNN
-F 1 "GND" H 2255 1977 50  0000 C CNN
-F 2 "" H 2250 2150 50  0001 C CNN
-F 3 "" H 2250 2150 50  0001 C CNN
-	1    2250 2150
+P 2800 2000
+F 0 "#PWR0103" H 2800 1750 50  0001 C CNN
+F 1 "GND" H 2805 1827 50  0000 C CNN
+F 2 "" H 2800 2000 50  0001 C CNN
+F 3 "" H 2800 2000 50  0001 C CNN
+	1    2800 2000
 	1    0    0    -1
 $EndComp
-Wire Wire Line
-	2250 2150 2250 2000
 $Comp
 L Device:R R3
@@
 Wire Wire Line
 	2800 1700 2800 2000
-Wire Wire Line
-	2800 2000 2250 2000
-Connection ~ 2250 2000
-Wire Wire Line
-	2250 2000 2250 1900
 NoConn ~ 2450 1400
 NoConn ~ 2450 1500
